File: Motor_Driver_ClearanceIssues2.brd (EAGLE design)
At the start: 127 x 76.2 mm, 88 parts

Commit message: board 2 almost done
Parts:
- moved C20 0.37 mm to (51.7, 24.1)
- moved R10 0.23 mm to (56.9, 16.5)
Routing:
- net GND: track 142.7 -> 185.3 mm, vias 6 -> 7
- net N$127: track 0.00 -> 37.6 mm, vias 0 -> 4
- net AGND: track 87.2 -> 116.6 mm, vias 5 -> 6
- net N$126: track 0.00 -> 25.0 mm, vias 0 -> 4
- net DGND: track 210.6 -> 233.7 mm, vias 9 -> 10
- net VCC: track 194.3 -> 178.2 mm, vias 6 -> 24
- net H3_VS: track 123.6 -> 117.5 mm, vias 21 -> 31
- net N$124: track 0.00 -> 4.01 mm
- net GAIN: track 63.0 -> 66.6 mm
- net N$17: track 14.6 -> 12.2 mm
- net H3_LOW: track 38.8 -> 37.0 mm
- net N$19: track 60.6 -> 59.4 mm
- net N$29: track 16.9 -> 15.8 mm
- net N$21: track 16.3 -> 15.7 mm
- net GL_C: track 51.5 -> 51.0 mm
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