File: Motor_Driver - Copy.brd (EAGLE design)
At the start: 100 x 50 mm, 74 parts, among them T1 TEENSY_3.1_ALL_PINS

Commit message: made minor changes starting to route board
Parts:
- removed D3, D4: SMAJ45CA-E3/61, SparkFun-DiscreteSemi:SMA-DIODE
- added R10, R11, R12, R13: 100R, adafruit:R0603
- added R7, R8, R9: 0, adafruit:R0603
- C1, C15, C16, C17, C18, C2, C27, C3: device adafruit:C0603 -> adafruit:C0805
- R26, R27, R28, R29, R30, R31: device adafruit:R0603 -> adafruit:R0805
- moved C25 87.1 mm to (-34.4, -2.54), turned to 0 degrees
- moved R28 58.7 mm to (14.8, 12.7), turned to 180 degrees
- moved R5 54.8 mm to (37.9, 19.1), flipped to the bottom, turned to 180 degrees
- moved R1 53.5 mm to (36.8, 31.8), flipped to the bottom, turned to 180 degrees
- moved R3 52.6 mm to (37.8, 23.5), flipped to the bottom, turned to 180 degrees
- moved C22 51.5 mm to (16.4, 6.35), flipped to the bottom, turned to 90 degrees
- moved R30 47.7 mm to (14.8, 10.5), turned to 180 degrees
- moved R26 47.5 mm to (18.1, 16.8), turned to 180 degrees
- moved C24 41.9 mm to (22.5, 6.35), flipped to the bottom
- moved T1 37.9 mm to (-27.0, 21.4), turned to 0 degrees
- moved C4 37.2 mm to (36.4, 13.0), flipped to the top
- moved U$15 34.8 mm to (51.3, 8.73), flipped to the bottom
- moved R6 33.1 mm to (37.9, 19.1), flipped to the top
- moved U$18 31.5 mm to (43.0, 12.2), turned to 0 degrees
- moved U$17 28.5 mm to (31.3, 12.2), turned to 0 degrees
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Connections:
- new net EN_GATE: T1.7, U$7.P$16
- new net N$11: C5.2, R13.1, U$7.P$30
- new net N$25: R12.2, U$17.P$1
- new net N$33: R11.2, U$18.P$2
- new net N$9: R10.2, U$18.P$1
- net GND: no longer D3.A, D4.A
- net H1_LOW: now also R8.2, R9.2
- net H3_LOW: now also R7.2
- net N$2: now also R9.1
- net N$22: now also R10.1; no longer U$18.P$1
- net N$23: now also R11.1; no longer U$18.P$2
- net N$24: now also R12.1; no longer U$17.P$1
- net N$3: now also R8.1
- net N$31: now also R13.2; no longer C5.2, U$7.P$30
- net N$6: now also R7.1
- net VCC: no longer D3.C, D4.C
Routing:
- net H1_VS: track 3.09 -> 79.6 mm, vias 8 -> 21
- net H2_VS: track 5.30 -> 75.3 mm, vias 8 -> 21
- net H3_VS: track 3.32 -> 71.5 mm, vias 8 -> 21
- net H1_LOW: track 0.00 -> 58.4 mm, vias 0 -> 1
- net H3_LOW: track 0.00 -> 56.0 mm, vias 0 -> 2
- net N$5: track 0.00 -> 55.9 mm, vias 0 -> 1
- net N$1: track 0.00 -> 43.6 mm, vias 0 -> 3
- net N$4: track 0.00 -> 41.8 mm, vias 0 -> 1
- net VCC: track 130.8 -> 90.9 mm, vias 2 -> 9
- net +5V: track 0.00 -> 37.3 mm, vias 0 -> 1
- net N$6: track 0.00 -> 33.7 mm, vias 0 -> 1
- net N$2: track 0.00 -> 26.5 mm, vias 0 -> 1
- net N$3: track 0.00 -> 26.5 mm, vias 0 -> 1
- net N$23: track 0.00 -> 18.8 mm
- net N$22: track 0.00 -> 13.2 mm
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- added copper zone on layer 1, net AGND
- added copper zone on layer 1, net VCC
- removed copper zone on layer 16, net DGND
- removed copper zone on layer 16, net H1_LOW
- removed copper zone on layer 16, net H1_VS
- removed copper zone on layer 16, net H2_VS
- removed copper zone on layer 16, net H3_LOW
- removed copper zone on layer 16, net H3_VS
Other:
- board size 100 x 50 mm -> 85.4 x 49.4 mm
- board text added: "*"
- board text added: "GND"
- board text added: "IND"
- board text added: "PWM"
- board text added: "PWRCAPS"
- board text added: "RX"
- board text added: "TX"
- board text added: "VCC"
