File: Motor_Driver.sch (EAGLE design)
At the start: 78 parts, among them T1 TEENSY_3.1_ALL_PINS

Commit message: made minor changes starting to route board
Parts:
- removed R10, R11, R12, R13: 100R, adafruit:R-US_R0603
- removed R7, R8, R9: 0, adafruit:R-US_R0603
- added C25: 0.015uF, adafruit:C-USC0603
- added D3, D4: SMAJ45CA-E3/61, SparkFun-DiscreteSemi:MBRA140
- C1, C15, C16, C17, C18, C2, C27, C3: device adafruit:C-USC0805 -> adafruit:C-USC0603
- R26, R27, R28, R29, R30, R31: device adafruit:R-US_R0805 -> adafruit:R-US_R0603
Connections:
- removed net +3.3V: T1.3.3V
- removed net +3V3: U$11.2
- removed net EN_GATE: T1.7/RX3, U$7.EN_GATE
- removed net N$11: C5.2, R13.1, U$7.SP2
- removed net N$25: R12.2, U$17.P$1
- removed net N$33: R11.2, U$18.P$2
- removed net N$9: R10.2, U$18.P$1
- removed net REF: U$7.REF
- new net N$30: C25.1, U$7.SS_TR
- new net REF3.3: T1.3.3V, U$11.2, U$7.REF
- net DGND: no longer C6.2, C7.2, R21.1
- net GND: now also C25.2, C6.2, C7.2, D3.A, D4.A, R21.1
- net H1_LOW: no longer R8.2, R9.2
- net H3_LOW: no longer R7.2
- net N$2: no longer R9.1
- net N$22: now also U$18.P$1; no longer R10.1
- net N$23: now also U$18.P$2; no longer R11.1
- net N$24: now also U$17.P$1; no longer R12.1
- net N$3: no longer R8.1
- net N$31: now also C5.2, U$7.SP2; no longer R13.2
- net N$6: no longer R7.1
- net VCC: now also D3.C, D4.C
