File: newone/Motor_Driver_Play.brd (EAGLE design)
At the start: 100 x 80 mm, 88 parts

Commit message: did stuff. So much of stuff
Parts:
- removed CTRL, SENS: 22-23-2041, con-molex:22-23-2041
- removed CURR: 22-23-2051, con-molex:22-23-2051
- removed M: 22-23-2081, con-molex:22-23-2081
- removed TEMP: 22-23-2021, con-molex:22-23-2021
- added U$8: STM32F4V_100PIN_GENERIC, stm32f4:LQFP100
- moved PT2 75.6 mm to (29.4, 7.62), turned to 270 degrees
- moved C27 57.4 mm to (4.60, 37.8), flipped to the top
- moved R32 57.1 mm to (4.76, 33.5), flipped to the top
- moved PT1 54.8 mm to (37.5, 47.5), turned to 270 degrees
- moved C25 52.2 mm to (2.70, 46.2), flipped to the top, turned to 90 degrees
- moved C26 47.2 mm to (5.87, 44.0), flipped to the top, turned to 270 degrees
- moved U$11 42.5 mm to (2.70, 42.4), flipped to the top, turned to 90 degrees
- moved U$10 33.9 mm to (12.7, 44.3), flipped to the top, turned to 270 degrees
- moved C9 33.5 mm to (21.7, 37.8), flipped to the top, turned to 90 degrees
- moved JP2 25.8 mm to (18.1, 36.5), turned to 270 degrees
- moved JP3 24.1 mm to (13.8, 36.5), turned to 270 degrees
- moved U$18 23.8 mm to (56.0, 32.2), flipped to the bottom, turned to 90 degrees
- moved JP4 22.6 mm to (9.84, 36.5), turned to 270 degrees
- moved C23 18.1 mm to (58.6, 41.3), turned to 90 degrees
- moved C12 18.1 mm to (43.7, 41.3), turned to 270 degrees
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Connections:
- net AGND: now also U$8.PA6; no longer CURR.5, SENS.4
- net DC_CAL: now also U$8.PE12; no longer CURR.4
- net DGND: now also U$8.PB11; no longer CTRL.4, M.1, TEMP.1
- net EN_GATE: now also U$8.PE11; no longer M.2
- net FAULT: now also U$8.PE13; no longer CTRL.2
- net H1: now also U$8.PE10; no longer M.3
- net H2: now also U$8.PE8; no longer M.5
- net H3: now also U$8.PB1; no longer M.7
- net L1: now also U$8.PE9; no longer M.4
- net L2: now also U$8.PE7; no longer M.6
- net L3: now also U$8.PB0; no longer M.8
- net OCTW: now also U$8.PE14; no longer CTRL.3
- net PWRGD: now also U$8.PE15; no longer CTRL.1
- net REF: now also U$8.PC5; no longer CURR.3
- net SENS1: now also U$8.PA3; no longer SENS.3
- net SENS2: now also U$8.PA4; no longer SENS.2
- net SENS3: now also U$8.PA5; no longer SENS.1
- net SO1: now also U$8.PC4; no longer CURR.2
- net SO2: now also U$8.PA7; no longer CURR.1
- net TEMP: now also U$8.PB10; no longer TEMP.2
Routing:
- net DGND: track 110.0 -> 6.30 mm, vias 1 -> 4
- net VCC: track 84.6 -> 38.6 mm, vias 0 -> 2
- net GND: track 45.0 -> 0.00 mm, vias 1 -> 16
- net AGND: track 31.0 -> 0.00 mm, vias 2 -> 0
- net H3_LOW: track 42.9 -> 13.1 mm, vias 1 -> 0
- net TEMP: track 54.3 -> 27.5 mm
- net +5V: track 74.7 -> 53.2 mm, vias 5 -> 1
- net DC_CAL: track 27.6 -> 9.53 mm, vias 1 -> 0
- net FAULT: track 26.0 -> 11.6 mm, vias 1 -> 0
- net SO2: track 22.9 -> 8.94 mm, vias 1 -> 0
- net EN_GATE: track 22.8 -> 8.94 mm
- net M_PWM: track 33.1 -> 19.2 mm, vias 0 -> 1
- net SENS1: track 22.5 -> 8.65 mm
- net SO1: track 22.3 -> 8.94 mm, vias 1 -> 0
- net REF: track 21.9 -> 8.94 mm, vias 1 -> 0
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- added copper zone on layer 1, net AGND
- added copper zone on layer 1, net DGND
- added copper zone on layer 1, net GND
- added copper zone on layer 16, net GND
Other:
- board size 100 x 80 mm -> 97.8 x 50.8 mm

Commit message: work damnit
Parts:
- moved U$12 39.7 mm to (57.9, 41.6), flipped to the bottom, turned to 90 degrees
- moved C22 33.5 mm to (25.9, 4.76)
- moved U$13 29.5 mm to (57.9, 23.8), flipped to the bottom, turned to 90 degrees
- moved C24 23.8 mm to (32.1, 4.76), turned to 90 degrees
- moved U$18 22.5 mm to (45.1, 12.5), turned to 0 degrees
- moved C23 16.1 mm to (44.3, 33.8)
- moved C21 12.1 mm to (46.5, 33.8)
- moved C11 10.7 mm to (37.5, 39.4)
- moved C12 10.3 mm to (52.7, 36.4), turned to 0 degrees
- moved C20 8.94 mm to (48.7, 33.8)
- moved R11 7.75 mm to (46.8, 13.3), turned to 90 degrees
- moved C19 7.33 mm to (44.3, 39.1), turned to 270 degrees
- moved R27 6.62 mm to (22.4, 18.1), turned to 180 degrees
- moved R31 6.62 mm to (17.6, 13.5), turned to 0 degrees
- moved R26 6.19 mm to (22.4, 16.0)
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Connections:
- net SENS1: now also U$8.PA5; no longer U$8.PA3
- net SENS3: now also U$8.PA3; no longer U$8.PA5
Routing:
- net H1_VS: track 8.65 -> 33.0 mm, vias 0 -> 2
- net H2_VS: track 10.7 -> 32.5 mm, vias 0 -> 2
- net H3_VS: track 11.0 -> 32.2 mm, vias 0 -> 2
- net H3_LOW: track 13.1 -> 29.1 mm, vias 0 -> 1
- net N$25: track 0.00 -> 7.75 mm, vias 0 -> 1
- net N$6: track 0.00 -> 6.05 mm
- net SENS3: track 5.42 -> 8.65 mm
- net SENS1: track 8.65 -> 5.42 mm
- net N$23: track 15.3 -> 18.5 mm
- net VCC: track 38.6 -> 35.5 mm, vias 2 -> 3
- net N$11: track 7.60 -> 5.56 mm
- net N$22: track 14.4 -> 13.2 mm
- net N$24: track 8.94 -> 7.77 mm
- net N$2: track 5.96 -> 5.16 mm
- net GL_A: track 4.29 -> 5.09 mm
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- added copper zone on layer 1, net VCC

Commit message: things happened. Board mostly done
Parts:
- R1, R2, R3, R4, R5, R6: value 4.7K -> 1
- R7, R8, R9: value 39K -> 0
- U$8: value STM32F4V_100PIN_GENERIC -> STM32F4R_64PIN_FOXCAR; device stm32f4:LQFP100 -> stm32f4:LQFP64
- moved U$15 50.0 mm to (49.4, 8.73), flipped to the bottom
- moved U$12 39.9 mm to (79.9, 8.26), flipped to the top
- moved U$16 37.3 mm to (49.8, 24.6), flipped to the bottom
- moved U$5 34.2 mm to (60.5, 8.26)
- moved U$6 34.2 mm to (69.4, 8.26)
- moved U$1 33.5 mm to (60.5, 41.0)
- moved U$2 33.5 mm to (69.4, 41.0)
- moved U$14 33.2 mm to (79.9, 41.0)
- moved U$13 21.8 mm to (79.7, 24.9), flipped to the top
- moved R13 21.6 mm to (27.6, 15.4), turned to 270 degrees
- moved U$4 17.0 mm to (60.5, 24.9), flipped to the top
- moved R29 16.1 mm to (6.35, 15.9), turned to 90 degrees
- moved R31 14.5 mm to (3.33, 15.7), turned to 90 degrees
- moved R27 13.0 mm to (9.53, 15.9), turned to 90 degrees
- moved R28 12.7 mm to (9.68, 12.7)
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Connections:
- net AGND: now also U$8.22; no longer U$8.PA6
- net DC_CAL: now also U$8.43; no longer U$8.PE12
- net DGND: now also U$8.53; no longer U$8.PB11
- net EN_GATE: now also U$8.42; no longer U$8.PE11
- net FAULT: now also U$8.44; no longer U$8.PE13
- net H1: now also U$8.41; no longer U$8.PE10
- net H2: now also U$8.39; no longer U$8.PE8
- net H3: now also U$8.37; no longer U$8.PB1
- net L1: now also U$8.40; no longer U$8.PE9
- net L2: now also U$8.38; no longer U$8.PE7
- net L3: now also U$8.36; no longer U$8.PB0
- net OCTW: now also U$8.45; no longer U$8.PE14
- net PWRGD: now also U$8.51; no longer U$8.PE15
- net REF: now also U$8.35; no longer U$8.PC5
- net SENS1: now also U$8.21; no longer U$8.PA5
- net SENS2: now also U$8.20; no longer U$8.PA4
- net SENS3: now also U$8.17; no longer U$8.PA3
- net SO1: now also U$8.34; no longer U$8.PC4
- net SO2: now also U$8.33; no longer U$8.PA7
- net TEMP: now also U$8.52; no longer U$8.PB10
Routing:
- net N$5: track 0.00 -> 56.2 mm, vias 0 -> 1
- net VCC: track 35.5 -> 86.8 mm, vias 3 -> 9
- net H1_VS: track 33.0 -> 81.4 mm, vias 2 -> 21
- net H2_VS: track 32.5 -> 78.6 mm, vias 2 -> 21
- net H1_LOW: track 13.7 -> 58.8 mm
- net N$1: track 0.00 -> 44.2 mm, vias 0 -> 3
- net N$4: track 0.00 -> 42.4 mm, vias 0 -> 1
- net H3_VS: track 32.2 -> 74.3 mm, vias 2 -> 21
- net H3_LOW: track 29.1 -> 57.5 mm, vias 1 -> 2
- net N$6: track 6.05 -> 34.3 mm, vias 0 -> 1
- net N$3: track 0.00 -> 27.1 mm, vias 0 -> 1
- net N$2: track 5.16 -> 27.1 mm
- net TEMP: track 27.5 -> 17.9 mm
- net N$9: track 0.00 -> 7.38 mm, vias 0 -> 1
- net N$33: track 0.00 -> 6.25 mm, vias 0 -> 1
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- added copper zone on layer 1, net H1_VS
- added copper zone on layer 1, net H2_VS
- added copper zone on layer 1, net H3_VS
Other:
- board size 97.8 x 50.8 mm -> 83.2 x 49.3 mm

Commit message: mostly done, w/ initial gerber files
Parts:
- added C28, C29, C30, C31, C32, C33, C34: 2.2uf, SparkFun-Capacitors:0603-CAP
- added C35, C36: 15pf, SparkFun-Capacitors:0603-CAP
- added C37: 0.1uf, SparkFun-Capacitors:0603-CAP
- added SV1: (no value), con-lsta:FE06
- added U$9: CRYSTAL-GROUNDED, SparkFun-FreqCtrl:CRYSTAL-SMD-5X3
- moved U$18 4.29 mm to (43.0, 12.2)
- moved U$17 4.29 mm to (31.3, 12.2)
- moved R31 3.97 mm to (7.30, 15.7)
- moved R29 3.81 mm to (10.2, 16.0)
- moved R27 3.81 mm to (13.3, 15.9)
- moved C22 3.70 mm to (16.4, 6.35)
- moved C24 3.70 mm to (22.5, 6.35)
- moved PT2 3.65 mm to (20.6, 10.0), turned to 180 degrees
- moved R26 3.49 mm to (16.5, 16.8)
- moved R28 3.33 mm to (13.0, 12.7)
- moved R30 3.33 mm to (13.0, 10.5)
- moved R32 3.02 mm to (6.99, 32.1)
- moved U$8 3.02 mm to (10.2, 24.3)
- moved R11 2.86 mm to (43.3, 13.0)
- moved C1 2.54 mm to (37.5, 29.2)
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Connections:
- new net N$32: C28.1, U$8.19
- new net N$34: C29.1, U$8.32
- new net N$35: C30.1, U$8.48
- new net N$36: C31.1, U$8.64
- new net N$37: C32.1, U$8.13
- new net N$38: C33.1, U$8.31
- new net N$39: C34.1, U$8.47
- new net N$40: C35.2, U$8.5, U$9.1
- new net N$41: C36.2, U$8.6, U$9.3
- new net NRST: C37.1, SV1.5, U$8.7
- new net SWCLK: SV1.2, U$8.49
- new net SWDIO: SV1.4, U$8.46
- net AGND: no longer R27.1, R29.1, R31.1
- net GND: now also C28.2, C29.2, C30.2, C31.2, C32.2, C33.2, C34.2, C35.1, C36.1, C37.2, R27.1, R29.1, R31.1, SV1.3, U$9.2, U$9.4
- net VCC: now also SV1.1
Routing:
- net SWCLK: track 0.00 -> 29.3 mm, vias 0 -> 1
- net SWDIO: track 0.00 -> 23.2 mm, vias 0 -> 1
- net VCC: track 86.8 -> 103.9 mm
- net NRST: track 0.00 -> 13.4 mm
- net GND: track 0.00 -> 11.8 mm, vias 27 -> 30
- net N$41: track 0.00 -> 6.56 mm, vias 0 -> 1
- net N$36: track 0.00 -> 5.48 mm, vias 0 -> 1
- net N$40: track 0.00 -> 5.38 mm, vias 0 -> 1
- net N$38: track 0.00 -> 4.53 mm, vias 0 -> 1
- net N$35: track 0.00 -> 4.18 mm, vias 0 -> 1
- net N$39: track 0.00 -> 2.98 mm, vias 0 -> 1
- net N$37: track 0.00 -> 2.63 mm, vias 0 -> 1
- net N$32: track 0.00 -> 2.61 mm, vias 0 -> 1
- net N$34: track 0.00 -> 2.48 mm, vias 0 -> 1
- net N$31: track 5.84 -> 7.58 mm
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Other:
- board size 83.2 x 49.3 mm -> 85.4 x 49.3 mm

Commit message: everything burns
Parts:
- added D3, D4, D5, D6: (no value), SparkFun-LED:LED-0603
- added JP1: USART, SparkFun-Connectors:1X04
- added R33: 10k, adafruit:R0603
- added R34: 120R, adafruit:R0603
- added R35, R36, R37, R38: 100R, adafruit:R0603
- added U$19: CAN_6P6C, Shell2015:CAN_6P6C
- added U1: MCP2551, SparkFun-DigitalIC:SO08
- SV1: device con-lsta:FE06 -> con-lstb:MA06-1
- moved C37 4.75 mm to (3.02, 26.4), turned to 90 degrees
- moved SV1 3.57 mm to (5.24, 8.41)
- moved R31 1.91 mm to (9.13, 15.2)
- moved R28 1.83 mm to (14.8, 12.7)
- moved R29 1.83 mm to (12.0, 16.0)
- moved R30 1.83 mm to (14.8, 10.5)
- moved R27 1.67 mm to (15.0, 15.9)
- moved R26 1.59 mm to (18.1, 16.8)
- moved C36 1.46 mm to (8.81, 23.9)
- moved C32 1.37 mm to (8.81, 20.4)
- moved PT2 1.35 mm to (22.0, 10.0)
- moved C28 1.33 mm to (9.53, 17.5), turned to 90 degrees
- moved C35 0.71 mm to (4.92, 30.1)
- moved C30 0.63 mm to (11.6, 28.6)
- moved U$9 0.48 mm to (5.00, 27.0)
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Connections:
- new net CAN1_RX: U$8.61, U1.4
- new net CAN1_TX: U$8.62, U1.1
- new net N$42: R33.1, U1.8
- new net N$43: R34.1, U$19.P$3, U1.7
- new net N$44: R34.2, U$19.P$5, U1.6
- new net N$45: D3.A, U$8.8
- new net N$46: D4.A, U$8.9
- new net N$47: D5.A, U$8.10
- new net N$48: D6.A, U$8.11
- new net N$49: D6.C, R38.1
- new net N$50: D5.C, R37.1
- new net N$51: D4.C, R36.1
- new net N$52: D3.C, R35.1
- new net RX: JP1.3, U$8.59
- new net TX: JP1.4, U$8.58
- net +5V: now also U$19.P$2, U1.3
- net GND: now also JP1.2, R33.2, R35.2, R36.2, R37.2, R38.2, U$19.P$4, U1.2
- net VCC: now also JP1.1
Routing:
- net N$43: track 0.00 -> 85.7 mm, vias 0 -> 1
- net N$44: track 0.00 -> 82.6 mm
- net +5V: track 49.2 -> 104.4 mm, vias 1 -> 2
- net RX: track 0.00 -> 30.9 mm, vias 0 -> 1
- net TX: track 0.00 -> 28.7 mm, vias 0 -> 1
- net CAN1_RX: track 0.00 -> 12.3 mm, vias 0 -> 3
- net N$48: track 0.00 -> 9.50 mm, vias 0 -> 1
- net CAN1_TX: track 0.00 -> 9.46 mm, vias 0 -> 1
- net GND: track 11.8 -> 20.5 mm, vias 30 -> 32
- net N$47: track 0.00 -> 7.02 mm, vias 0 -> 1
- net NRST: track 13.4 -> 18.8 mm
- net SWCLK: track 29.3 -> 34.0 mm, vias 1 -> 2
- net N$42: track 0.00 -> 4.24 mm
- net N$46: track 0.00 -> 3.04 mm, vias 0 -> 1
- net N$45: track 0.00 -> 2.80 mm, vias 0 -> 1
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Other:
- board size 85.4 x 49.3 mm -> 85.4 x 49.4 mm
