File: newone/Motor_Driver_Play.brd (EAGLE design)
At the start: 85.4 x 49.4 mm, 109 parts, among them U1 MCP2551

Commit message: Added silkscreen to top/bottom layer
Other:
- board text added: "*"
- board text added: "GAIN"
- board text added: "GND"
- board text added: "IND"
- board text added: "OC"
- board text added: "PWM"
- board text added: "PWRCAPS"
- board text added: "RX"
- board text added: "TX"
- board text added: "VCC"
Changed lines of the file:
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@@
 <layer number="23" name="tOrigins" color="15" fill="1" visible="yes" active="yes"/>
 <layer number="24" name="bOrigins" color="15" fill="1" visible="yes" active="yes"/>
-<layer number="25" name="tNames" color="7" fill="1" visible="no" active="yes"/>
-<layer number="26" name="bNames" color="7" fill="1" visible="no" active="yes"/>
+<layer number="25" name="tNames" color="7" fill="1" visible="yes" active="yes"/>
+<layer number="26" name="bNames" color="7" fill="1" visible="yes" active="yes"/>
 <layer number="27" name="tValues" color="7" fill="1" visible="no" active="yes"/>
 <layer number="28" name="bValues" color="7" fill="1" visible="no" active="yes"/>
@@
 <wire x1="85.4075" y1="49.276" x2="0" y2="49.276" width="0" layer="20"/>
 <wire x1="0" y1="49.276" x2="0" y2="-0.079375" width="0" layer="20"/>
+<text x="26.51125" y="30.00375" size="1.778" layer="25" rot="MR0">*</text>
+<text x="3.571875" y="0.9525" size="1.27" layer="25" rot="R90">VCC</text>
+<text x="12.620625" y="10.556875" size="1.27" layer="25" rot="R180">TX</text>
+<text x="12.938125" y="7.9375" size="1.27" layer="25" rot="R180">RX</text>
+<text x="14.366875" y="5.3975" size="1.27" layer="25" rot="R180">GND</text>
+<text x="14.208125" y="2.778125" size="1.27" layer="25" rot="R180">VCC</text>
+<text x="11.826875" y="35.08375" size="1.27" layer="25" rot="R90">GAIN</text>
+<text x="15.954375" y="35.956875" size="1.27" layer="25" rot="R90">OC</text>
+<text x="20.0025" y="34.925" size="1.27" layer="25" rot="R90">PWM</text>
+<text x="15.24" y="33.734375" size="1.27" layer="25" rot="R180">VCC</text>
+<text x="10.556875" y="33.258125" size="1.27" layer="25">*</text>
+<text x="14.525625" y="33.258125" size="1.27" layer="25">*</text>
+<text x="18.89125" y="33.258125" size="1.27" layer="25">*</text>
+<text x="11.43" y="41.036875" size="1.27" layer="25">GND</text>
+<text x="38.4175" y="41.43375" size="1.27" layer="25">PWRCAPS</text>
+<text x="24.13" y="1.349375" size="1.27" layer="25" rot="MR0">PWRCAPS</text>
+<text x="37.94125" y="45.323125" size="1.27" layer="26" rot="MR0">IND</text>
+<text x="38.25875" y="3.4925" size="1.016" layer="25" rot="R270">VCC</text>
+<text x="36.195" y="3.413125" size="1.016" layer="25" rot="R270">GND</text>
 </plain>
 <attributes>
@@
 </class>
 </classes>
-<designrules name="APCircuits *">
+<designrules name="ITEADstudio_DRC">
 <description language="de">&lt;b&gt;EAGLE Design Rules&lt;/b&gt;
 &lt;p&gt;
@@
 <element name="D1" library="nxp" package="SOD123W" value="PMEG6020ER,115" x="33.17875" y="35.71875" rot="MR180"/>
 <element name="D2" library="SparkFun-DiscreteSemi" package="SMA-DIODE" value="SMAJ5.0A" x="25.24125" y="43.18" rot="R180"/>
-<element name="JP2" library="pinhead" package="1X03" value="M_PWM" x="17.4625" y="37.62375" rot="R270"/>
-<element name="JP3" library="pinhead" package="1X03" value="M_OC" x="13.17625" y="37.62375" rot="R270"/>
-<element name="JP4" library="pinhead" package="1X03" value="GAIN" x="9.2075" y="37.62375" rot="R270"/>
+<element name="JP2" library="pinhead" package="1X03" value="M_PWM" x="17.4625" y="37.62375" smashed="yes" rot="R270">
+<attribute name="VALUE" x="14.2875" y="41.43375" size="1.27" layer="27" rot="R270"/>
+</element>
+<element name="JP3" library="pinhead" package="1X03" value="M_OC" x="13.17625" y="37.62375" smashed="yes" rot="R270">
+<attribute name="VALUE" x="10.00125" y="41.43375" size="1.27" layer="27" rot="R270"/>
+</element>
+<element name="JP4" library="pinhead" package="1X03" value="GAIN" x="9.2075" y="37.62375" smashed="yes" rot="R270">
+<attribute name="VALUE" x="6.0325" y="41.43375" size="1.27" layer="27" rot="R270"/>
+</element>
 <element name="L1" library="bourne" package="SDR0805" value="22uH" x="33.9725" y="41.11625" rot="MR180"/>
 <element name="PT1" library="SparkFun-Passives" package="2PT_GND_TIE" value="2PT_GND_TIE" x="33.416875" y="47.14875" rot="R270"/>
@@
 <element name="C35" library="SparkFun-Capacitors" package="0603-CAP" value="15pf" x="4.92125" y="30.083125" rot="MR0"/>
 <element name="C36" library="SparkFun-Capacitors" package="0603-CAP" value="15pf" x="8.810625" y="23.891875" rot="MR0"/>
-<element name="SV1" library="con-lstb" package="MA06-1" value="" x="5.23875" y="8.41375" rot="R90">
+<element name="SV1" library="con-lstb" package="MA06-1" value="" x="5.23875" y="8.41375" smashed="yes" rot="R90">
 <attribute name="MF" value="" x="5.23875" y="8.41375" size="1.778" layer="27" rot="R90" display="off"/>
 <attribute name="OC_NEWARK" value="unknown" x="5.23875" y="8.41375" size="1.778" layer="27" rot="R90" display="off"/>
 <attribute name="MPN" value="" x="5.23875" y="8.41375" size="1.778" layer="27" rot="R90" display="off"/>
 <attribute name="OC_FARNELL" value="unknown" x="5.23875" y="8.41375" size="1.778" layer="27" rot="R90" display="off"/>
+<attribute name="VALUE" x="8.15975" y="5.87375" size="1.27" layer="27" ratio="10" rot="R90"/>
 </element>
 <element name="C37" library="SparkFun-Capacitors" package="0603-CAP" value="0.1uf" x="3.01625" y="26.431875" rot="R90"/>
@@
 <attribute name="PARTNO" value="553-2258-ND" x="21.11375" y="22.70125" size="1.778" layer="27" display="off"/>
 </element>
-<element name="JP1" library="SparkFun-Connectors" package="1X04" value="USART" x="8.89" y="2.2225" rot="R90"/>
+<element name="JP1" library="SparkFun-Connectors" package="1X04" value="USART" x="8.89" y="2.2225" smashed="yes" rot="R90">
+<attribute name="VALUE" x="12.065" y="0.9525" size="1.27" layer="27" rot="R90"/>
+</element>
 </elements>
 <signals>
@@
 <wire x1="6.850625" y1="28.1375" x2="6.889375" y2="28.09875" width="0.4064" layer="16"/>
 <wire x1="6.889375" y1="28.09875" x2="8.41375" y2="28.09875" width="0.4064" layer="16"/>
+<wire x1="8.41375" y1="28.09875" x2="8.6925" y2="27.66125" width="0" layer="19" extent="16-16"/>
+<wire x1="15.24" y1="16.295" x2="15.001875" y2="14.875" width="0" layer="19" extent="1-16"/>
+<wire x1="11.985625" y1="15.03375" x2="13.17625" y2="16.295" width="0" layer="19" extent="1-16"/>
+<wire x1="31.83921875" y1="23.49125" x2="29.05125" y2="23.33625" width="0" layer="19" extent="1-1"/>
+<wire x1="57.42305" y1="28.73375" x2="50.165" y2="34.29" width="0" layer="19" extent="16-16"/>
 </signal>
 <signal name="SO2">
@@
 <wire x1="24.13" y1="44.235" x2="24.13" y2="45.56125" width="0.4064" layer="16"/>
 <contactref element="U$8" pad="53"/>
+<wire x1="12.235" y1="28.86375" x2="16.1925" y2="29.5275" width="0" layer="19" extent="1-1"/>
+<wire x1="6.82625" y1="31.1175" x2="12.235" y2="28.86375" width="0" layer="19" extent="1-1"/>
+<wire x1="24.13" y1="39.74375" x2="21.2725" y2="36.04125" width="0" layer="19" extent="1-16"/>
 </signal>
 <signal name="+5V">
@@
 <wire x1="53.0225" y1="6.0325" x2="51.91125" y2="6.985" width="0" layer="19" extent="1-1"/>
 <wire x1="61.11875" y1="8.255" x2="53.0225" y2="8.09625" width="0" layer="19" extent="1-1"/>
+<wire x1="31.83921875" y1="30.99125" x2="38.89375" y2="34.89625" width="0" layer="19" extent="1-1"/>
 </signal>
 <signal name="N$18">
