File: newone/Motor_Driver_Play.sch (EAGLE design)
At the start: 88 parts

Commit message: did stuff. So much of stuff
Parts:
- removed CTRL, SENS: 22-23-2041, con-molex:22-23-2041
- removed CURR: 22-23-2051, con-molex:22-23-2051
- removed M: 22-23-2081, con-molex:22-23-2081
- removed TEMP: 22-23-2021, con-molex:22-23-2021
- added U$8: STM32F4V_100PIN_GENERIC, stm32f4:STM32F4V_100PIN_GENERIC
Connections:
- net AGND: now also U$8.PA6; no longer CURR-5.S, SENS-4.S
- net DC_CAL: now also U$8.PE12; no longer CURR-4.S
- net DGND: now also U$8.PB11; no longer CTRL-4.S, M-1.S, TEMP-1.S
- net EN_GATE: now also U$8.PE11; no longer M-2.S
- net FAULT: now also U$8.PE13; no longer CTRL-2.S
- net H1: now also U$8.PE10; no longer M-3.S
- net H2: now also U$8.PE8; no longer M-5.S
- net H3: now also U$8.PB1; no longer M-7.S
- net L1: now also U$8.PE9; no longer M-4.S
- net L2: now also U$8.PE7; no longer M-6.S
- net L3: now also U$8.PB0; no longer M-8.S
- net OCTW: now also U$8.PE14; no longer CTRL-3.S
- net PWRGD: now also U$8.PE15; no longer CTRL-1.S
- net REF: now also U$8.PC5; no longer CURR-3.S
- net SENS1: now also U$8.PA3; no longer SENS-3.S
- net SENS2: now also U$8.PA4; no longer SENS-2.S
- net SENS3: now also U$8.PA5; no longer SENS-1.S
- net SO1: now also U$8.PC4; no longer CURR-2.S
- net SO2: now also U$8.PA7; no longer CURR-1.S
- net TEMP: now also U$8.PB10; no longer TEMP-2.S
Other:
- note removed: "Control Connector"
- note removed: "Motor Control Connector"
- moved on the sheet: C19, C20, C21, C22

Commit message: work damnit
Connections:
- net SENS1: now also U$8.PA5; no longer U$8.PA3
- net SENS3: now also U$8.PA3; no longer U$8.PA5
Changed lines of the file:
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@@
 <setting verticaltext="up"/>
 </settings>
-<grid distance="0.05" unitdist="inch" unit="inch" style="lines" multiple="1" display="yes" altdistance="0.01" altunitdist="inch" altunit="inch"/>
+<grid distance="0.05" unitdist="inch" unit="inch" style="lines" multiple="1" display="no" altdistance="0.01" altunitdist="inch" altunit="inch"/>
 <layers>
 <layer number="1" name="Top" color="4" fill="1" visible="no" active="no"/>
@@
 </segment>
 <segment>
-<pinref part="U$8" gate="G$1" pin="PA3"/>
-<wire x1="374.65" y1="26.67" x2="370.84" y2="26.67" width="0.1524" layer="91"/>
-<label x="370.84" y="26.67" size="1.016" layer="95" rot="R180" xref="yes"/>
+<pinref part="U$8" gate="G$1" pin="PA5"/>
+<wire x1="374.65" y1="21.59" x2="370.84" y2="21.59" width="0.1524" layer="91"/>
+<label x="370.84" y="21.59" size="1.016" layer="95" rot="R180" xref="yes"/>
 </segment>
 </net>
@@
 </segment>
 <segment>
-<pinref part="U$8" gate="G$1" pin="PA5"/>
-<wire x1="374.65" y1="21.59" x2="370.84" y2="21.59" width="0.1524" layer="91"/>
-<label x="370.84" y="21.59" size="1.016" layer="95" rot="R180" xref="yes"/>
-</segment>
-</net>
+<pinref part="U$8" gate="G$1" pin="PA3"/>
+<wire x1="374.65" y1="26.67" x2="370.84" y2="26.67" width="0.1524" layer="91"/>
+<label x="370.84" y="26.67" size="1.016" layer="95" rot="R180" xref="yes"/>
+</segment>
+</net>

Commit message: things happened. Board mostly done
Parts:
- R1, R2, R3, R4, R5, R6: value 4.7K -> 1
- R7, R8, R9: value 39K -> 0
- U$8: value STM32F4V_100PIN_GENERIC -> STM32F4R_64PIN_FOXCAR; device stm32f4:STM32F4V_100PIN_GENERIC -> stm32f4:STM32F4R_64PIN_FOXCAR
Connections:
- net DC_CAL: now also U$8.PA10; no longer U$8.PE12
- net DGND: now also U$8.PC12; no longer U$8.PB11
- net EN_GATE: now also U$8.PA9; no longer U$8.PE11
- net FAULT: now also U$8.PA11; no longer U$8.PE13
- net H1: now also U$8.PA8; no longer U$8.PE10
- net H2: now also U$8.PC8; no longer U$8.PE8
- net H3: now also U$8.PC6; no longer U$8.PB1
- net L1: now also U$8.PC9; no longer U$8.PE9
- net L2: now also U$8.PC7; no longer U$8.PE7
- net L3: now also U$8.PB15; no longer U$8.PB0
- net OCTW: now also U$8.PA12; no longer U$8.PE14
- net PWRGD: now also U$8.PC10; no longer U$8.PE15
- net REF: now also U$8.PB14; no longer U$8.PC5
- net SO1: now also U$8.PB13; no longer U$8.PC4
- net SO2: now also U$8.PB12; no longer U$8.PA7
- net TEMP: now also U$8.PC11; no longer U$8.PB10

Commit message: mostly done, w/ initial gerber files
Parts:
- added C28, C29, C30, C31, C32, C33, C34: 2.2uf, SparkFun-Capacitors:CAP0603-CAP
- added C35, C36: 15pf, SparkFun-Capacitors:CAP0603-CAP
- added C37: 0.1uf, SparkFun-Capacitors:CAP0603-CAP
- added SV1: (no value), con-lsta:FE06-1
- added U$9: CRYSTAL-GROUNDED, SparkFun-FreqCtrl:CRYSTAL-GROUNDED
Connections:
- new net N$32: C28.1, U$8.VDD1
- new net N$34: C29.1, U$8.VDD2
- new net N$35: C30.1, U$8.VDD3
- new net N$36: C31.1, U$8.VDD4
- new net N$37: C32.1, U$8.VDDA
- new net N$38: C33.1, U$8.VCAP1
- new net N$39: C34.1, U$8.VCAP2
- new net N$40: C35.2, U$8.PH0, U$9.2
- new net N$41: C36.2, U$8.PH1, U$9.1
- new net NRST: C37.1, SV1.5, U$8.NRST
- new net SWCLK: SV1.2, U$8.PA14
- new net SWDIO: SV1.4, U$8.PA13
- net AGND: no longer R27.1, R29.1, R31.1
- net GND: now also C28.2, C29.2, C30.2, C31.2, C32.2, C33.2, C34.2, C35.1, C36.1, C37.2, R27.1, R29.1, R31.1, SV1.3, U$9.3
- net VCC: now also SV1.1

Commit message: everything burns
Parts:
- added D3, D4, D5, D6: (no value), SparkFun-LED:LED0603
- added JP1: USART, SparkFun-Connectors:M04PTH
- added R33: 10k, adafruit:R-US_R0603
- added R34: 120R, adafruit:R-US_R0603
- added R35, R36, R37, R38: 100R, adafruit:R-US_R0603
- added U$19: CAN_6P6C, Shell2015:CAN_6P6C
- added U1: MCP2551, SparkFun-DigitalIC:MCP2551
- SV1: device con-lsta:FE06-1 -> con-lstb:MA06-1
Connections:
- new net CAN1_RX: U$8.PB8, U1.RXD
- new net CAN1_TX: U$8.PB9, U1.TXD
- new net N$42: R33.1, U1.RS
- new net N$43: R34.1, U$19.CANH, U1.CANH
- new net N$44: R34.2, U$19.CANL, U1.CANL
- new net N$45: D3.A, U$8.PC0
- new net N$46: D4.A, U$8.PC1
- new net N$47: D5.A, U$8.PC2
- new net N$48: D6.A, U$8.PC3
- new net N$49: D6.C, R38.1
- new net N$50: D5.C, R37.1
- new net N$51: D4.C, R36.1
- new net N$52: D3.C, R35.1
- new net RX: JP1.3, U$8.PB7
- new net TX: JP1.4, U$8.PB6
- net +5V: now also U$19.VCC, U1.VDD
- net GND: now also JP1.2, R33.2, R35.2, R36.2, R37.2, R38.2, U$19.GND, U1.VSS
- net VCC: now also JP1.1
